Commit message: driving_bot

File: src/mobile_bot/urdf/robot.urdf.xacro (robot description, xacro)
@@ -2,3 +2,4 @@
 <robot xmlns:xacro="http://www.ros.org/wiki/xacro" name="rd_bot_1.0M"  >
     <xacro:include filename="$(find mobile_bot)/urdf/robot_core.xacro"/>
+   <xacro:include filename="$(find mobile_bot)/urdf/gazebo_control.xacro"/>
 </robot>

File: src/mobile_bot/urdf/robot_core.xacro (robot description, xacro)
@@ -1,125 +1,133 @@
 <?xml version="1.0"?>
-<robot xmlns:xacro="http://www.ros.org/wiki/xacro">
-  <xacro:include filename="$(find mobile_bot)/urdf/inertial_macros.xacro"/>
-<!-- COLOUR -->
-<material name="white">
- <color rgba="1 1 1 1"/>
- </material>
-<material name="orange">
-    <color rgba="1 0.3 0.1 1"/>
-</material>
-<material name="blue">
-    <color rgba="0.2 0.2 1.0 1"/>
-</material>
-<material name="black">
-     <color rgba="0.0 0.0 0.0 1.0"/>
-</material>
-<!-- WORLD LINK -->
-<link name="world">
-</link>
-<!-- CHASIS WORLD JOINT -->
-<joint name="chasis_joint" type="fixed">
-    <parent link="world"/>
-    <child link="chasis"/>
-    <origin xyz="-0.1 0.0 0.0" rpy="0.0 0.0 0.0"/>
-</joint>
-<!-- CHASIS LINK -->
-<link name="chasis">
-    <xacro:inertial_box mass="0.5" x="0.4" y="0.3" z="0.15">
-    <origin xyz="0.15 0.0 0.075" rpy="0 0 0"/>
-     </xacro:inertial_box>
-    <visual>
-        <origin xyz="0.15 0.0 0.075" rpy="0.0 0.0 0.0"/>
-        <geometry>
-            <box size="0.4 0.3 0.15"/>
-        </geometry>
-        <material name="white"/>
-    </visual>
-    <collision>
-        <origin xyz="0.15 0.0 0.075" rpy="0.0 0.0 0.0"/>
-        <geometry>
-            <box size="0.4 0.3 0.15"/>
-        </geometry>
-    </collision>
-</link>
- <!-- LEFT WHEEL MACRO -->
-<xacro:macro name="left_wheel" params="name x y z">
-    <link name="${name}">
-    <visual>
-        <geometry>
-          <mesh filename="package://mobile_bot/Mesh/left_tire.stl" scale="0.0025 0.0025 0.0025"/>
-        </geometry>
-        <material name="LightGrey">
-            <color rgba="0.7 0.7 0.7 1.0"/>
-        </material>
-    </visual>
-    <collision>
-        <geometry>
-        <mesh filename="package://mobile_bot/Mesh/left_tire.stl" scale="0.0025 0.0025 0.0025"/>
-        </geometry>
-    </collision>
-    <xacro:inertial_cylinder mass="0.1" length="0.04" radius="0.08">
-    <origin xyz="0 0 0" rpy="0 0 0"/>
-     </xacro:inertial_cylinder>
-</link>
-<joint name="${name}_base_joint" type="continuous">
-    <origin xyz="${x} ${y} 0.0" rpy="0 0 0"/>
-    <parent link="world"/>
-    <child link="${name}"/>
-    <axis xyz="0 1 0"/>
-</joint>
-</xacro:macro>
-<!-- RIGHT WHEEL MACRO -->
-<xacro:macro name="right_wheel" params="name x y z">
-    <link name="${name}">
-    <visual>
-        <geometry>
-          <mesh filename="package://mobile_bot/Mesh/right_tire.stl" scale="0.0025 0.0025 0.0025"/>
-        </geometry>
-        <material name="LightGrey">
-            <color rgba="0.7 0.7 0.7 1.0"/>
-        </material>
-    </visual>
-    <collision>
-        <geometry>
-        <mesh filename="package://mobile_bot/Mesh/right_tire.stl" scale="0.0025 0.0025 0.0025"/>
-        </geometry>
-    </collision>
-   <xacro:inertial_cylinder mass="0.1" length="0.04" radius="0.08">
-    <origin xyz="0 0 0" rpy="0 0 0"/>
-     </xacro:inertial_cylinder>
-</link>
-<joint name="${name}_base_joint" type="continuous">
-    <origin xyz="${x} ${y} 0.0" rpy="0 0 0"/>
-    <parent link="world"/>
-    <child link="${name}"/>
-    <axis xyz="0 1 0"/>
-</joint>
-</xacro:macro>
- <!-- LEFT WHEEL -->
-<xacro:left_wheel name="left_wheel" x="0.0" y="0.175" z="0.0"/>
- <!-- RIGHT WHEEL -->
- <xacro:right_wheel name="right_wheel" x="0.0" y="-0.175" z="0.0"/>
-<!-- CASTER wHEEL LINK -->
-<joint name="caster_wheel" type="fixed">
- <parent link="chasis"/>
- <child link="caster"/>
- <origin xyz="0.24 0.0 0.0" rpy="0.0 0.0 0.0"/>
-</joint>
-<link name="caster">
-<visual>
-    <geometry>
-        <sphere radius="0.07"/>
-    </geometry>
-    <material name="black"/>
-</visual>
-<collision>
-     <geometry>
-        <sphere radius="0.07"/>
-    </geometry>
-</collision>
-<xacro:inertial_sphere mass="0.1" radius="0.07">
-    <origin xyz="0 0 0" rpy="0 0 0"/>
-     </xacro:inertial_sphere>
-</link>
+<robot xmlns:xacro="http://www.ros.org/wiki/xacro" >
+    <xacro:include filename="inertial_macros.xacro"/>
+    <material name="white">
+        <color rgba="1 1 1 1" />
+    </material>
+    <material name="orange">
+        <color rgba="1 0.3 0.1 1"/>
+    </material>
+    <material name="blue">
+        <color rgba="0.2 0.2 1 1"/>
+    </material>
+    <material name="black">
+        <color rgba="0 0 0 1"/>
+    </material>
+    <!-- BASE LINK -->
+    <link name="base_link">
+    </link>
+    <!-- CHASSIS LINK -->
+    <joint name="chassis_joint" type="fixed">
+        <parent link="base_link"/>
+        <child link="chassis"/>
+        <origin xyz="-0.1 0 0"/>
+    </joint>
+    <link name="chassis">
+        <visual>
+            <origin xyz="0.15 0 0.075"/>
+            <geometry>
+                <box size="0.3 0.3 0.15"/>
+            </geometry>
+            <material name="white"/>
+        </visual>
+        <collision>
+            <origin xyz="0.15 0 0.075"/>
+            <geometry>
+                <box size="0.3 0.3 0.15"/>
+            </geometry>
+        </collision>
+        <xacro:inertial_box mass="0.5" x="0.3" y="0.3" z="0.15">
+            <origin xyz="0.15 0 0.075" rpy="0 0 0"/>
+        </xacro:inertial_box>
+    </link>
+    <gazebo reference="chassis">
+      <material>
+        Gazebo/Orange
+      </material>
+    </gazebo>
+    <!-- LEFT WHEEL LINK -->
+    <joint name="left_wheel_joint" type="continuous">
+        <parent link="base_link"/>
+        <child link="left_wheel"/>
+        <origin xyz="0 0.175 0" rpy="-${pi/2} 0 0" />
+        <axis xyz="0 0 1"/>
+    </joint>
+    <link name="left_wheel">
+        <visual>
+            <geometry>
+                <cylinder radius="0.05" length="0.04"/>
+            </geometry>
+            <material name="blue"/>
+        </visual>
+        <collision>
+            <geometry>
+                <cylinder radius="0.05" length="0.04"/>
+            </geometry>
+        </collision>
+        <xacro:inertial_cylinder mass="0.1" length="0.04" radius="0.05">
+            <origin xyz="0 0 0" rpy="0 0 0"/>
+        </xacro:inertial_cylinder>
+    </link>
+    <gazebo reference="left_wheel">
+      <material>
+        Gazebo/Black
+      </material>
+    </gazebo>
+    <!-- RIGHT WHEEL LINK -->
+    <joint name="right_wheel_joint" type="continuous">
+        <parent link="base_link"/>
+        <child link="right_wheel"/>
+        <origin xyz="0 -0.175 0" rpy="${pi/2} 0 0" />
+        <axis xyz="0 0 -1"/>
+    </joint>
+    <link name="right_wheel">
+        <visual>
+            <geometry>
+                <cylinder radius="0.05" length="0.04"/>
+            </geometry>
+            <material name="blue"/>
+        </visual>
+        <collision>
+            <geometry>
+                <cylinder radius="0.05" length="0.04"/>
+            </geometry>
+        </collision>
+        <xacro:inertial_cylinder mass="0.1" length="0.04" radius="0.05">
+            <origin xyz="0 0 0" rpy="0 0 0"/>
+        </xacro:inertial_cylinder>
+    </link>
+   <gazebo reference="right_wheel">
+      <material>
+        Gazebo/Black
+      </material>
+    </gazebo>
+    <!-- CASTER WHEEL LINK -->
+    <joint name="caster_wheel_joint" type="fixed">
+        <parent link="chassis"/>
+        <child link="caster_wheel"/>
+        <origin xyz="0.24 0 0"/>
+    </joint>
+    <link name="caster_wheel">
+        <visual>
+            <geometry>
+                <sphere radius="0.05"/>
+            </geometry>
+            <material name="black"/>
+        </visual>
+        <collision>
+            <geometry>
+                <sphere radius="0.05"/>
+            </geometry>
+        </collision>
+        <xacro:inertial_sphere mass="0.1" radius="0.05">
+            <origin xyz="0 0 0" rpy="0 0 0"/>
+        </xacro:inertial_sphere>
+    </link>
+    <gazebo reference="caster_wheel">
+      <material>
+        Gazebo/White
+      </material>
+      <mu1 value="0.001"/>
+      <mu2 value="0.001"/>
+    </gazebo>
 </robot>
