Commit message: control and mapping

File: src/mobile_bot/urdf/lidar.xacro (robot description, xacro)
@@ -25,5 +25,5 @@
 <sensor name="laser" type="ray">
    <pose>0 0 0 0 0 0</pose>
-   <visualize>false</visualize>
+   <visualize>true</visualize>
     <update_rate>10</update_rate>
     <ray>

File: src/mobile_bot/urdf/robot_core.xacro (robot description, xacro)
@@ -17,4 +17,11 @@
     <link name="base_link">
     </link>
+<joint name="base_footprint_joint" type="fixed">
+        <parent link="base_link"/>
+        <child link="base_footprint"/>
+        <origin xyz="0 0 0"/>
+    </joint>
+<link name="base_footprint">
+    </link>
     <!-- CHASSIS LINK -->
     <joint name="chassis_joint" type="fixed">
@@ -29,5 +36,5 @@
                 <box size="0.3 0.3 0.15"/>
             </geometry>
-            <material name="white"/>
+            <material name="orange"/>
         </visual>
         <collision>
