Commit message: holiday

File: src/mobile_bot/urdf/camera.xacro (robot description, xacro)
@@ -4,5 +4,5 @@
     <parent link="chassis"/>
     <child link="camera_link"/>
-    <origin xyz="0.305 0.0 0.08" rpy="0.0 0.0 0.0"/>
+    <origin xyz="0.305 0.0 0.08" rpy="0.0 0.018 0.0"/>
 </joint>
 <link name="camera_link">
@@ -25,5 +25,5 @@
   <pose>0 0 0 0 0 0</pose>
       <always_on>true</always_on>
-      <visualize>true</visualize>
+      <visualize>false</visualize>
       <updateRate>10</updateRate>
       <camera>

File: src/mobile_bot/urdf/camera_depth.xacro (robot description, xacro)
@@ -1,10 +1,10 @@
 <?xml version="1.0"?>
 <robot xmlns:xacro="http://www.ros.org/wiki/xacro">
-<joint name="camera_joint" type="fixed">
+<joint name="camera_depth_joint" type="fixed">
     <parent link="chassis"/>
-    <child link="camera_link"/>
+    <child link="camera_depth_link"/>
     <origin xyz="0.305 0.0 0.08" rpy="0.0 0.0 0.0"/>
 </joint>
-<link name="camera_link">
+<link name="camera_depth_link">
       <visual>
             <geometry>
@@ -14,12 +14,12 @@
         </visual>
 </link>
-<joint name="camera_opticcal_joint" type="fixed">
-    <parent link="camera_link"/>
-    <child link="camera_optical_link"/>
+<joint name="camera_optical_depth_joint" type="fixed">
+    <parent link="camera_depth_link"/>
+    <child link="camera_optical_depth_link"/>
     <origin xyz="0 0.0 0.0" rpy="${-pi/2} 0.0 ${-pi/2}"/>
 </joint>
-<link name="camera_optical_link">
+<link name="camera_optical_depth_link">
 </link>
-<gazebo reference="camera_link">
+<gazebo reference="camera_depth_link">
   <sensor type="depth" name="camera_depth">
   <pose>0 0 0 0 0 0</pose>
@@ -39,10 +39,10 @@
           </clip>
       </camera>
- <plugin name="camera_controller" filename="libgazebo_ros_openni_kinect.so">
+ <plugin name="camera_depth_controller" filename="libgazebo_ros_openni_kinect.so">
           <baseline>0.2</baseline>
         <alwaysOn>true</alwaysOn>
         <updateRate>30.0</updateRate>
         <cameraName>camera</cameraName>
-        <frameName>camera_optical_link</frameName>
+        <frameName>camera_optical_depth_link</frameName>
          <imageTopicName>rgb/image_raw</imageTopicName>
         <depthImageTopicName>depth/image_raw</depthImageTopicName>

File: src/mobile_bot/urdf/robot.urdf.xacro (robot description, xacro)
@@ -1,9 +1,8 @@
 <?xml version="1.0"?>
 <robot xmlns:xacro="http://www.ros.org/wiki/xacro" name="rd_bot_1.0M"  >
-<xacro:include filename="$(find turtlebot3_description)/urdf/turtlebot3_burger.gazebo.xacro"/>
     <xacro:include filename="$(find mobile_bot)/urdf/robot_core.xacro"/>
    <xacro:include filename="$(find mobile_bot)/urdf/gazebo_control.xacro"/>
     <xacro:include filename="$(find mobile_bot)/urdf/lidar.xacro"/>
-    <!-- <xacro:include filename="$(find mobile_bot)/urdf/camera.xacro"/> -->
+    <xacro:include filename="$(find mobile_bot)/urdf/camera.xacro"/>
     <xacro:include filename="$(find mobile_bot)/urdf/camera_depth.xacro"/>
 </robot>
